Commit message: dof_forceを入力に追加、ランダムに機体がジャンプするようにした

File: hoge.urdf (robot description, URDF)
Before this commit: robot hoge, 13 links, 12 joints
Links:
- link base_link: mass 10 -> 12; geometry visual box size=0.5 0.4 0.2
- link head_link: geometry visual box size=0.2 0.25 0.15
Joints:
- joint leg0_joint_1: origin xyz=0.2 0.2 0 rpy=0 0 0 -> xyz=0.15 0.1 0 rpy=0 0 0
- joint leg1_joint_1: origin xyz=0.2 -0.2 0 rpy=0 0 0 -> xyz=0.15 -0.1 0 rpy=0 0 0
- joint leg2_joint_1: origin xyz=-0.3 0.2 0 rpy=0 0 0 -> xyz=-0.2 0.1 0 rpy=0 0 0
- joint leg3_joint_1: origin xyz=-0.3 -0.2 0 rpy=0 0 0 -> xyz=-0.2 -0.1 0 rpy=0 0 0
