Commit message: モデルをさらに小さく&フレーミーに変更

File: framy.urdf (robot description, URDF)
Before this commit: robot hoge, 13 links, 12 joints
Links:
- removed link neck_link
- added link ear_left_link; visual box size=0.05 0.1 0.1
- added link ear_right_link; visual box size=0.05 0.1 0.1
- added link nose_link; visual box size=0.1 0.1 0.05
- added link nose_tip_link; visual box size=0.05 0.1 0.02
- added link tail_link; visual box size=0.1 0.1 0.05
- link base_link: mass 12 -> 8; geometry visual box size=0.4 0.3 0.2
- link eye_left_link: geometry visual cylinder length=0.02 radius=0.02
- link eye_right_link: geometry visual cylinder length=0.02 radius=0.02
- link head_link: geometry visual box size=0.2 0.2 0.2
- link leg0_link_2: mass 1 -> 2; geometry collision box size=0.05 0.05 0.25; visual box size=0.05 0.05 0.25
- link leg1_link_2: mass 1 -> 2; geometry collision box size=0.05 0.05 0.25; visual box size=0.05 0.05 0.25
- link leg2_link_2: mass 1 -> 2; geometry collision box size=0.05 0.05 0.25; visual box size=0.05 0.05 0.25
- link leg3_link_2: mass 1 -> 2; geometry collision box size=0.05 0.05 0.25; visual box size=0.05 0.05 0.25
Joints:
- removed joint neck
- added joint ear_left: type fixed, parent head_link, child ear_left_link, origin xyz=-0.02 0.05 0.15000000000000002 rpy=0 0 0
- added joint ear_right: type fixed, parent head_link, child ear_right_link, origin xyz=-0.02 -0.05 0.15000000000000002 rpy=0 0 0
- added joint nose: type fixed, parent head_link, child nose_link, origin xyz=0.07 0 0 rpy=0 0 0
- added joint nose_tip: type fixed, parent nose_link, child nose_tip_link, origin xyz=0.1 0 0.05 rpy=0 0 0
- added joint tail: type fixed, parent base_link, child tail_link, origin xyz=-0.15000000000000002 0 0.1 rpy=0 0 0
- joint eye_left: origin xyz=0.1 -0.08 0.075 rpy=0 1.5707963267948966 0 -> xyz=0.1 -0.05 0.1 rpy=0 1.5707963267948966 0
- joint eye_right: origin xyz=0.1 0.08 0.075 rpy=0 1.5707963267948966 0 -> xyz=0.1 0.05 0.1 rpy=0 1.5707963267948966 0
- joint head: origin xyz=0 0 0.1 rpy=0 0 0 -> xyz=0.25000000000000006 0 0.05 rpy=0 0 0; parent neck_link -> base_link
- joint leg0_joint_1: origin xyz=0.15 0.1 0 rpy=0 0 0 -> xyz=0.1 0.08 0 rpy=0 0 0
- joint leg1_joint_1: origin xyz=0.15 -0.1 0 rpy=0 0 0 -> xyz=0.1 -0.08 0 rpy=0 0 0
- joint leg2_joint_1: origin xyz=-0.2 0.1 0 rpy=0 0 0 -> xyz=-0.15 0.08 0 rpy=0 0 0
- joint leg3_joint_1: origin xyz=-0.2 -0.1 0 rpy=0 0 0 -> xyz=-0.15 -0.08 0 rpy=0 0 0

Commit message: 足の先端にcylinderを追加

File: framy.urdf (robot description, URDF)
Before this commit: robot framy, 17 links, 16 joints
Links:
- added link leg0_link_3, mass 0.3; collision cylinder length=0.05 radius=0.03; visual cylinder length=0.05 radius=0.03
- added link leg1_link_3, mass 0.3; collision cylinder length=0.05 radius=0.03; visual cylinder length=0.05 radius=0.03
- added link leg2_link_3, mass 0.3; collision cylinder length=0.05 radius=0.03; visual cylinder length=0.05 radius=0.03
- added link leg3_link_3, mass 0.3; collision cylinder length=0.05 radius=0.03; visual cylinder length=0.05 radius=0.03
- link base_link: mass 8 -> 10.8
- link leg0_link_2: mass 2 -> 1
- link leg1_link_2: mass 2 -> 1
- link leg2_link_2: mass 2 -> 1
- link leg3_link_2: mass 2 -> 1
Joints:
- added joint leg0_joint_3: type fixed, parent leg0_link_2, child leg0_link_3, origin xyz=0 0 -0.25 rpy=0 0 0
- added joint leg1_joint_3: type fixed, parent leg1_link_2, child leg1_link_3, origin xyz=0 0 -0.25 rpy=0 0 0
- added joint leg2_joint_3: type fixed, parent leg2_link_2, child leg2_link_3, origin xyz=0 0 -0.25 rpy=0 0 0
- added joint leg3_joint_3: type fixed, parent leg3_link_2, child leg3_link_3, origin xyz=0 0 -0.25 rpy=0 0 0
- joint leg0_joint_1: origin xyz=0.1 0.08 0 rpy=0 0 0 -> xyz=0.1 0.08 0.05 rpy=0 0 0
- joint leg1_joint_1: origin xyz=0.1 -0.08 0 rpy=0 0 0 -> xyz=0.1 -0.08 0.05 rpy=0 0 0
- joint leg2_joint_1: origin xyz=-0.15 0.08 0 rpy=0 0 0 -> xyz=-0.15 0.08 0.05 rpy=0 0 0
- joint leg3_joint_1: origin xyz=-0.15 -0.08 0 rpy=0 0 0 -> xyz=-0.15 -0.08 0.05 rpy=0 0 0

Commit message: 重さ0はだめらしい

File: framy.urdf (robot description, URDF)
Before this commit: robot framy, 21 links, 20 joints
Links:
- link base_link: mass 10.8 -> 19.08
- link ear_left_link: mass None -> 0.001
- link ear_right_link: mass None -> 0.001
- link eye_left_link: mass None -> 0.001
- link eye_right_link: mass None -> 0.001
- link head_link: mass None -> 0.001
- link leg0_link_1: mass 1 -> 0.1
- link leg0_link_2: mass 1 -> 0.1
- link leg0_link_3: mass 0.3 -> 0.03
- link leg1_link_1: mass 1 -> 0.1
- link leg1_link_2: mass 1 -> 0.1
- link leg1_link_3: mass 0.3 -> 0.03
- link leg2_link_1: mass 1 -> 0.1
- link leg2_link_2: mass 1 -> 0.1
- link leg2_link_3: mass 0.3 -> 0.03
- link leg3_link_1: mass 1 -> 0.1
- link leg3_link_2: mass 1 -> 0.1
- link leg3_link_3: mass 0.3 -> 0.03
- link nose_link: mass None -> 0.001
- link nose_tip_link: mass None -> 0.001
- link tail_link: mass None -> 0.001

Commit message: かなり不安定だけど動くようになったっぽい

File: framy.urdf (robot description, URDF)
Before this commit: robot framy, 21 links, 20 joints
Links:
- link base_link: mass 19.08 -> 4.0
- link leg0_link_1: mass 0.1 -> 1.5
- link leg0_link_2: mass 0.1 -> 2
- link leg0_link_3: mass 0.03 -> 0.5
- link leg1_link_1: mass 0.1 -> 1.5
- link leg1_link_2: mass 0.1 -> 2
- link leg1_link_3: mass 0.03 -> 0.5
- link leg2_link_1: mass 0.1 -> 1.5
- link leg2_link_2: mass 0.1 -> 2
- link leg2_link_3: mass 0.03 -> 0.5
- link leg3_link_1: mass 0.1 -> 1.5
- link leg3_link_2: mass 0.1 -> 2
- link leg3_link_3: mass 0.03 -> 0.5

Commit message: 膝にcylinderを追加

File: framy.urdf (robot description, URDF)
Before this commit: robot framy, 21 links, 20 joints
Links:
- added link leg0_link_4, mass 0.001; visual cylinder length=0.05 radius=0.025
- added link leg1_link_4, mass 0.001; visual cylinder length=0.05 radius=0.025
- added link leg2_link_4, mass 0.001; visual cylinder length=0.05 radius=0.025
- added link leg3_link_4, mass 0.001; visual cylinder length=0.05 radius=0.025
Joints:
- added joint leg0_joint_4: type fixed, parent leg0_link_2, child leg0_link_4, origin xyz=0 0 0 rpy=0 0 0
- added joint leg1_joint_4: type fixed, parent leg1_link_2, child leg1_link_4, origin xyz=0 0 0 rpy=0 0 0
- added joint leg2_joint_4: type fixed, parent leg2_link_2, child leg2_link_4, origin xyz=0 0 0 rpy=0 0 0
- added joint leg3_joint_4: type fixed, parent leg3_link_2, child leg3_link_4, origin xyz=0 0 0 rpy=0 0 0

Commit message: 5本足にする

File: framy.urdf (robot description, URDF)
Before this commit: robot framy, 25 links, 24 joints
Links:
- added link longleg_link_0, mass 0.5; visual box size=0.05 0.05 0.25
- added link longleg_link_1, mass 0.5; visual box size=0.05 0.05 0.25
- added link longleg_link_10, mass 0.5; visual box size=0.05 0.05 0.25
- added link longleg_link_11, mass 0.5; collision box size=0.05 0.05 0.25; visual box size=0.05 0.05 0.25
- added link longleg_link_2, mass 0.5; visual box size=0.05 0.05 0.25
- added link longleg_link_3, mass 0.5; visual box size=0.05 0.05 0.25
- added link longleg_link_4, mass 0.5; visual box size=0.05 0.05 0.25
- added link longleg_link_5, mass 0.5; visual box size=0.05 0.05 0.25
- added link longleg_link_6, mass 0.5; visual box size=0.05 0.05 0.25
- added link longleg_link_7, mass 0.5; visual box size=0.05 0.05 0.25
- added link longleg_link_8, mass 0.5; visual box size=0.05 0.05 0.25
- added link longleg_link_9, mass 0.5; visual box size=0.05 0.05 0.25
- link base_link: mass 4.0 -> 7.6
- link leg0_link_1: mass 1.5 -> 0.5
- link leg0_link_2: mass 2 -> 1
- link leg0_link_3: mass 0.5 -> 0.1
- link leg1_link_1: mass 1.5 -> 0.5
- link leg1_link_2: mass 2 -> 1
- link leg1_link_3: mass 0.5 -> 0.1
- link leg2_link_1: mass 1.5 -> 0.5
- link leg2_link_2: mass 2 -> 1
- link leg2_link_3: mass 0.5 -> 0.1
- link leg3_link_1: mass 1.5 -> 0.5
- link leg3_link_2: mass 2 -> 1
- link leg3_link_3: mass 0.5 -> 0.1
Joints:
- added joint longleg_joint_0: type continuous, parent base_link, child longleg_link_0, origin xyz=0.125 0 0 rpy=0 0 0, axis 0 1 0
- added joint longleg_joint_1: type continuous, parent longleg_link_0, child longleg_link_1, origin xyz=0 0 -0.25 rpy=0 0 0, axis 0 1 0
- added joint longleg_joint_10: type continuous, parent longleg_link_9, child longleg_link_10, origin xyz=0 0 -0.25 rpy=0 0 0, axis 0 1 0
- added joint longleg_joint_11: type continuous, parent longleg_link_10, child longleg_link_11, origin xyz=0 0 -0.25 rpy=0 0 0, axis 0 1 0
- added joint longleg_joint_2: type continuous, parent longleg_link_1, child longleg_link_2, origin xyz=0 0 -0.25 rpy=0 0 0, axis 0 1 0
- added joint longleg_joint_3: type continuous, parent longleg_link_2, child longleg_link_3, origin xyz=0 0 -0.25 rpy=0 0 0, axis 0 1 0
- added joint longleg_joint_4: type continuous, parent longleg_link_3, child longleg_link_4, origin xyz=0 0 -0.25 rpy=0 0 0, axis 0 1 0
- added joint longleg_joint_5: type continuous, parent longleg_link_4, child longleg_link_5, origin xyz=0 0 -0.25 rpy=0 0 0, axis 0 1 0
- added joint longleg_joint_6: type continuous, parent longleg_link_5, child longleg_link_6, origin xyz=0 0 -0.25 rpy=0 0 0, axis 0 1 0
- added joint longleg_joint_7: type continuous, parent longleg_link_6, child longleg_link_7, origin xyz=0 0 -0.25 rpy=0 0 0, axis 0 1 0
- added joint longleg_joint_8: type continuous, parent longleg_link_7, child longleg_link_8, origin xyz=0 0 -0.25 rpy=0 0 0, axis 0 1 0
- added joint longleg_joint_9: type continuous, parent longleg_link_8, child longleg_link_9, origin xyz=0 0 -0.25 rpy=0 0 0, axis 0 1 0

Commit message: パラメーターをいじった

File: framy.urdf (robot description, URDF)
Before this commit: robot framy, 37 links, 36 joints
Links:
- link base_link: mass 7.6 -> 1.5999999999999996
- link leg0_link_1: mass 0.5 -> 1.0
- link leg0_link_2: mass 1 -> 2.0
- link leg1_link_1: mass 0.5 -> 1.0
- link leg1_link_2: mass 1 -> 2.0
- link leg2_link_1: mass 0.5 -> 1.0
- link leg2_link_2: mass 1 -> 2.0
- link leg3_link_1: mass 0.5 -> 1.0
- link leg3_link_2: mass 1 -> 2.0

Commit message: section2まで踏破

File: framy.urdf (robot description, URDF)
Before this commit: robot framy, 37 links, 36 joints
Links:
- link longleg_link_0: geometry collision box size=0.05 0.05 0.25; visual box size=0.05 0.05 0.25
- link longleg_link_1: geometry collision box size=0.05 0.05 0.25; visual box size=0.05 0.05 0.25
- link longleg_link_10: geometry collision box size=0.05 0.05 0.25; visual box size=0.05 0.05 0.25
- link longleg_link_2: geometry collision box size=0.05 0.05 0.25; visual box size=0.05 0.05 0.25
- link longleg_link_3: geometry collision box size=0.05 0.05 0.25; visual box size=0.05 0.05 0.25
- link longleg_link_4: geometry collision box size=0.05 0.05 0.25; visual box size=0.05 0.05 0.25
- link longleg_link_5: geometry collision box size=0.05 0.05 0.25; visual box size=0.05 0.05 0.25
- link longleg_link_6: geometry collision box size=0.05 0.05 0.25; visual box size=0.05 0.05 0.25
- link longleg_link_7: geometry collision box size=0.05 0.05 0.25; visual box size=0.05 0.05 0.25
- link longleg_link_8: geometry collision box size=0.05 0.05 0.25; visual box size=0.05 0.05 0.25
- link longleg_link_9: geometry collision box size=0.05 0.05 0.25; visual box size=0.05 0.05 0.25
